Commit message: fix urdf mesh origin. add lidar link. edit readme

File: src/asv_description/urdf/wamv_base.urdf (robot description, URDF)
Before this commit: robot wam-v, 2 links, 1 joints
Links:
- added link wamv/dummy_link_fix_mesh_origin, mass 180.0; collision box size=0.65 0.2 0.1; collision box size=0.65 0.2 0.1
- added link wamv/lidar_link
- link wamv/base_link: mass 180.0 -> None; geometry 
- link wamv/imu_link: mass 0.1 -> None
Joints:
- added joint fix_origin_joint: type fixed, parent wamv/base_link, child wamv/dummy_link_fix_mesh_origin, origin xyz=0 0 -0.36 rpy=0 0 0
- added joint lidar_joint: type fixed, parent wamv/base_link, child wamv/lidar_link, origin xyz=0.701 0 1.031 rpy=0 0 0
- joint imu_joint: origin xyz=1 0 1 rpy=0 0 0 -> xyz=0 0 0.944 rpy=0 0 0

Commit message: devcontainer forward display, camera link urdf

File: src/asv_description/urdf/wamv_base.urdf (robot description, URDF)
Before this commit: robot wam-v, 4 links, 3 joints
Links:
- added link wamv/camera_link
Joints:
- added joint camera_joint: type fixed, parent wamv/base_link, child wamv/camera_link, origin xyz=0.701 0 1.031 rpy=0 0 0

Commit message: bugged commit, see previous commit

File: src/asv_description/urdf/wamv_base.urdf (robot description, URDF)
Before this commit: robot wam-v, 5 links, 4 joints
Links:
- removed link wamv/base_link
- removed link wamv/camera_link
- removed link wamv/dummy_link_fix_mesh_origin
- removed link wamv/imu_link
- removed link wamv/lidar_link
- added link base_footprint
- added link base_link
- added link camera_link
- added link dummy_link_fix_mesh_origin, mass 180.0; collision box size=0.65 0.2 0.1; collision box size=0.65 0.2 0.1
- added link imu_link
- added link lidar_link
Joints:
- added joint footprint_joint: type fixed, parent base_link, child base_footprint, origin xyz=0.0 0 0.0 rpy=0 0 0
- joint camera_joint: child wamv/camera_link -> camera_link; parent wamv/base_link -> base_link
- joint fix_origin_joint: child wamv/dummy_link_fix_mesh_origin -> dummy_link_fix_mesh_origin; parent wamv/base_link -> base_link
- joint imu_joint: child wamv/imu_link -> imu_link; parent wamv/base_link -> base_link
- joint lidar_joint: child wamv/lidar_link -> lidar_link; parent wamv/base_link -> base_link
